Commit message: updates to description

File: osr_description/urdf/osr_description.urdf (robot description, URDF)
Before this commit: robot osr_description, 3 links, 2 joints
Joints:
- joint depth_camera_joint: origin xyz=1 0 1 rpy=0 0 3.14 -> xyz=0 0.14 0.45 rpy=0 0 3.14
- joint tracking_camera_joint: origin xyz=1 0 1 rpy=0 0 3.14 -> xyz=0 0.14 0.39 rpy=0 0 3.14

Commit message: Updates to urdf and json config

File: osr_description/urdf/osr_description.urdf (robot description, URDF)
Before this commit: robot osr_description, 3 links, 2 joints
Joints:
- joint depth_camera_joint: origin xyz=0 0.14 0.45 rpy=0 0 3.14 -> xyz=0.14 0 0.45 rpy=0 0 0
- joint tracking_camera_joint: origin xyz=0 0.14 0.39 rpy=0 0 3.14 -> xyz=0.14 0 0.39 rpy=0 0 0
